File: devices/GenericSensor/KiCad/GenericSensor_v1.sch (KiCad schematic (older format))
At the start: 25 parts, among them J1 Conn_01x06_Male, J2 Conn_01x09_Male, J3 Conn_01x04_Male, SW1 BOOT, SW2 RESET, U1 STM32L041K6Tx, U2 RFM95W-868S2, Y1 32KHz

Commit message: Small fixes for distance
Parts:
- renumbered SW1 to BOOT1, SW2 to RESET1
Changed lines of the file:
@@
 	4500 3650 4500 3800
 $Comp
-L Switch:SW_Push SW2
+L Switch:SW_Push RESET1
 U 1 1 5ECB7E79
 P 5050 3000
-F 0 "SW2" H 5050 3285 50  0000 C CNN
-F 1 "RESET" H 5050 3194 50  0000 C CNN
+F 0 "RESET1" H 5050 3200 50  0000 C CNN
+F 1 "RESET" H 5050 3194 50  0001 C CNN
 F 2 "Button_Switch_SMD:SW_SPST_TL3342" H 5050 3200 50  0001 C CNN
 F 3 "~" H 5050 3200 50  0001 C CNN
@@
 $EndComp
 $Comp
-L Switch:SW_Push SW1
+L Switch:SW_Push BOOT1
 U 1 1 5ECB9728
 P 4300 3200
-F 0 "SW1" H 4300 3485 50  0000 C CNN
-F 1 "BOOT" H 4300 3394 50  0000 C CNN
+F 0 "BOOT1" H 4300 3400 50  0000 C CNN
+F 1 "BOOT" H 4300 3394 50  0001 C CNN
 F 2 "Button_Switch_SMD:SW_SPST_TL3342" H 4300 3400 50  0001 C CNN
 F 3 "~" H 4300 3400 50  0001 C CNN
