File: devices/GenericSensor/KiCad/GenericSensor_v1.kicad_pcb (KiCad board)
At the start: 2 copper layers, 25 x 59.7 mm, 25 parts, among them J1 Conn_01x06_Male, J2 Conn_01x09_Male, J3 Conn_01x04_Male, SW1 BOOT, SW2 RESET, U1 STM32L041K6Tx, U2 RFM95W-868S2, Y1 32KHz

Commit message: Small fixes for distance
Parts:
- renumbered SW1 to BOOT, SW2 to RESET
Connections:
- J1 pad 4: SWCLK -> SWDIO
- J1 pad 5: SWDIO -> SWCLK
Other:
- board text added: "Generic Sensor 1.2 04.July.2020"
- board text removed: "Soil Sensor v2.1 07.06.2020"
