File: devices/GenericSensor/KiCad/GenericSensor_v2.kicad_pcb (KiCad board)
At the start: 2 copper layers, 25 x 59.7 mm, 35 parts, among them J1 Conn_01x06_Male, J2 Conn_01x09_Male, J3 Conn_01x04_Male, U1 STM32L041K6Tx, U2 RFM95W-868S2, Y1 32KHz

Commit message: refresh to latest libraries
Parts:
- J1: footprint Connector_PinSocket_2.54mm:PinSocket_1x06_P2.54mm_Vertical -> Connector_PinHeader_2.54mm:PinHeader_1x06_P2.54mm_Vertical
- J2: footprint Connector_PinSocket_2.54mm:PinSocket_1x09_P2.54mm_Vertical -> Connector_PinHeader_2.54mm:PinHeader_1x09_P2.54mm_Vertical
- J3: footprint Connector_PinSocket_2.54mm:PinSocket_2x02_P2.54mm_Vertical -> Connector_PinHeader_2.54mm:PinHeader_2x02_P2.54mm_Vertical
- moved J3 2.55 mm to (126.4, 39.6)
Connections:
- J3 pad 1: A9 -> A0
- J3 pad 2: A0 -> A9
- J3 pad 3: A8 -> A1
- J3 pad 4: A1 -> A8
- U2 pad 11: (no net) -> unconnected-(U2-Pad11)
- U2 pad 12: (no net) -> unconnected-(U2-Pad12)
- U2 pad 7: (no net) -> unconnected-(U2-Pad7)
Other:
- net class Default removed
