File: devices/SoilSensor/KiCad/SoilSensor_v2.kicad_pcb (KiCad board)
At the start: 2 copper layers, 24.9 x 143.8 mm, 28 parts, among them J1 Conn_01x06_Male, U2 RFM95W-868S2, U3 SoilSonde, Y1 32KHz

Commit message: Small revision -> 2.2
Parts:
- removed C3: 100 nF, Capacitor_SMD:C_0805_2012Metric
- removed R8: 10K, Resistor_SMD:R_0805_2012Metric
- removed REF** (x2): MountingHole_2.2mm_M2, MountingHole:MountingHole_2.2mm_M2
- added H1: MountingHole, MountingHole:MountingHole_2.2mm_M2, F.Cu at (146.5, 83.9)
- added H2: MountingHole, MountingHole:MountingHole_2.2mm_M2, F.Cu at (127.3, 41.0)
- FB1: footprint Resistor_SMD:R_1206_3216Metric -> Resistor_SMD:R_0805_2012Metric
- R1, R7: value 10K -> 12K
- R2: value 10M -> 2M2
- moved SW1 0.07 mm to (146.5, 48.3)
- moved SW2 0.05 mm to (146.5, 57.1)
- renumbered BOOT to SW1, RESET to SW2, STM32Lx to U1
Connections:
- U1 pad 15: Net-(U1-Pad15) -> (no net)
- U1 pad 18: Net-(U1-Pad18) -> (no net)
- U1 pad 19: Net-(U1-Pad19) -> (no net)
- U1 pad 27: Net-(U1-Pad27) -> (no net)
- U1 pad 28: Net-(U1-Pad28) -> (no net)
- U1 pad 29: Net-(U1-Pad29) -> (no net)
- U1 pad 6: Net-(U1-Pad6) -> (no net)
- U1 pad 7: Net-(U1-Pad7) -> (no net)
- U2 pad 11: Net-(U2-Pad11) -> (no net)
- U2 pad 12: Net-(U2-Pad12) -> (no net)
- U2 pad 7: Net-(U2-Pad7) -> (no net)
Routing:
- net +3V3: track 98.9 -> 95.4 mm, vias 3 -> 2
- net Net-(C4-Pad1): track 40.3 -> 37.7 mm, vias 3 -> 2
- net Net-(R7-Pad1): track 65.0 -> 63.4 mm
Other:
- board text added: "Soil Sensor v2.2 05 July 2020"
- board text removed: "Soil Sensor v2.1 07.06.2020"
