File: devices/SoilSensor/KiCad/SoilSensor_v2.sch (KiCad schematic (older format))
At the start: 26 parts, among them J1 Conn_01x06_Male, SW1 BOOT, SW2 RESET, U1 STM32L041K6Tx, U2 RFM95W-868S2, U3 SoilSonde, Y1 32KHz

Commit message: Small revision -> 2.2
Parts:
- removed C3: empty, Capacitor_SMD:C_0805_2012Metric, symbol Device:C
- removed R8: 12K, Resistor_SMD:R_0805_2012Metric, symbol Device:R
- added H1, H2: MountingHole, MountingHole:MountingHole_2.2mm_M2, symbol Mechanical:MountingHole
Connections:
- wire segments 47 -> 44
Changed lines of the file:
@@
 Sheet 1 1
 Title "Capacitive Soil Sensor for Lorawan"
-Date "2020-06-07"
-Rev "2.1"
+Date "2020-07-05"
+Rev "2.2"
 Comp ""
-Comment1 "BUG1: boot condensator should be connected to ground to avoid entering in bootloader at power on"
+Comment1 ""
 Comment2 ""
 Comment3 ""
@@
 	0    1    1    0
 $EndComp
-$Comp
-L Device:C C3
-U 1 1 5ECBAEA8
-P 4300 2750
-F 0 "C3" V 4048 2750 50  0000 C CNN
-F 1 "empty" V 4139 2750 50  0000 C CNN
-F 2 "Capacitor_SMD:C_0805_2012Metric" H 4338 2600 50  0001 C CNN
-F 3 "~" H 4300 2750 50  0001 C CNN
-	1    4300 2750
-	0    1    1    0
-$EndComp
-Wire Wire Line
-	4450 2750 4500 2750
-Wire Wire Line
-	4500 2750 4500 3200
 Connection ~ 4500 3200
 Wire Wire Line
@@
 Wire Wire Line
 	4100 3200 4100 2750
-Wire Wire Line
-	4100 2750 4150 2750
 $Comp
 L power:GND #PWR0104
@@
 	1    0    0    -1
 $EndComp
-Connection ~ 4100 2750
 Wire Wire Line
 	4800 3500 5250 3500
@@
 $EndComp
 $Comp
-L Device:R R8
-U 1 1 5ED83258
-P 5250 2450
-F 0 "R8" V 5250 2450 50  0000 C CNN
-F 1 "12K" V 5366 2450 50  0000 C CNN
-F 2 "Resistor_SMD:R_0805_2012Metric" V 5180 2450 50  0001 C CNN
-F 3 "~" H 5250 2450 50  0001 C CNN
-	1    5250 2450
-	-1   0    0    1
-$EndComp
-$Comp
-L power:+3.3V #PWR0117
-U 1 1 5ED84A32
-P 5250 2300
-F 0 "#PWR0117" H 5250 2150 50  0001 C CNN
-F 1 "+3.3V" H 5265 2473 50  0001 C CNN
-F 2 "" H 5250 2300 50  0001 C CNN
-F 3 "" H 5250 2300 50  0001 C CNN
-	1    5250 2300
-	1    0    0    -1
-$EndComp
-$Comp
 L Soil~Sensor:SoilSonde U3
 U 1 1 5EDF65A1
@@
 Wire Wire Line
 	4850 3000 4850 2600
-Connection ~ 5250 2600
 Wire Wire Line
 	6650 4500 6350 4500
 Wire Wire Line
 	5250 4100 4450 4100
+$Comp
+L Mechanical:MountingHole H1
+U 1 1 5F026DCA
+P 5500 5200
+F 0 "H1" H 5600 5246 50  0000 L CNN
+F 1 "MountingHole" H 5600 5155 50  0000 L CNN
+F 2 "MountingHole:MountingHole_2.2mm_M2" H 5500 5200 50  0001 C CNN
+F 3 "~" H 5500 5200 50  0001 C CNN
+	1    5500 5200
+	1    0    0    -1
+$EndComp
+$Comp
+L Mechanical:MountingHole H2
+U 1 1 5F027B85
+P 5500 5450
+F 0 "H2" H 5600 5496 50  0000 L CNN
+F 1 "MountingHole" H 5600 5405 50  0000 L CNN
+F 2 "MountingHole:MountingHole_2.2mm_M2" H 5500 5450 50  0001 C CNN
+F 3 "~" H 5500 5450 50  0001 C CNN
+	1    5500 5450
+	1    0    0    -1
+$EndComp
 $EndSCHEMATC
